Commit message: Updates in youbot urdf file (wheels)

File: youbot-team3/ros-pkg/youbot_model/urdf/youbot.urdf (robot description, URDF)
Before this commit: robot youbot, 6 links, 5 joints
Links:
- added link finger1_link; visual mesh filename=package://youbot_model/mesh/finger.stl
- added link finger2_link; visual mesh filename=package://youbot_model/mesh/finger.stl
- added link wheel_1_link; visual mesh filename=package://youbot_model/mesh/wheel.stl
- added link wheel_2_link; visual mesh filename=package://youbot_model/mesh/wheel.stl
- added link wheel_3_link; visual mesh filename=package://youbot_model/mesh/wheel.stl
- added link wheel_4_link; visual mesh filename=package://youbot_model/mesh/wheel.stl
Joints:
- added joint f1: type prismatic, parent link5, child finger1_link, origin xyz=-0.008 0.0 0.048, axis -1 0 0
- added joint f2: type prismatic, parent link5, child finger2_link, origin xyz=0.008 0.0 0.048 rpy=0 0 3.14, axis -1 0 0
- added joint w1: type continuous, parent base_link, child wheel_1_link, origin xyz=-0.158 -0.228 -0.053, axis 1 0 0
- added joint w2: type continuous, parent base_link, child wheel_2_link, origin xyz=0.158 -0.228 -0.053 rpy=0 3.14 0, axis 1 0 0
- added joint w3: type continuous, parent base_link, child wheel_3_link, origin xyz=0.158 0.228 -0.053, axis 1 0 0
- added joint w4: type continuous, parent base_link, child wheel_4_link, origin xyz=-0.158 0.228 -0.053 rpy=0 3.14 0, axis 1 0 0
